File: fuentesimetrica/fuentesimetrica.kicad_sch (KiCad schematic)
At the start: 15 parts, among them J1 terminal 3 pines, J2 Screw_Terminal_01x01, J3 Screw_Terminal_01x01, J4 Screw_Terminal_01x01, U1 uA7815, U2 L7915

Commit message: Agrego proyecto banco de R y nanoamperimetro, fuente simetrica
Parts:
- C1, C2: footprint Capacitor_THT:CP_Axial_L25.0mm_D10.0mm_P30.00mm_Horizontal -> Capacitor_THT:CP_Radial_D10.0mm_P2.50mm
- C3, C4: footprint Capacitor_THT:CP_Axial_L25.0mm_D10.0mm_P30.00mm_Horizontal -> Capacitor_THT:CP_Radial_Tantal_D4.5mm_P2.50mm
- C5, C6: footprint Capacitor_THT:CP_Axial_L25.0mm_D10.0mm_P30.00mm_Horizontal -> Capacitor_THT:CP_Radial_D4.0mm_P1.50mm
- D2: footprint (none) -> LED_THT:LED_D5.0mm_Horizontal_O1.27mm_Z3.0mm
- J2, J3, J4: footprint (none) -> TerminalBlock_MetzConnect:TerminalBlock_MetzConnect_360271_1x01_Horizontal_ScrewM3.0_Boxed
- R1: value R -> 220; footprint (none) -> Resistor_THT:R_Axial_DIN0411_L9.9mm_D3.6mm_P5.08mm_Vertical
- U1, U2: footprint (none) -> Package_TO_SOT_THT:TO-220F-3_Vertical
Connections:
- net 0 is gone; now on net GND: C1.2, C2.1, D2.1 (K), J3.1 (Pin_1)
- net GND: now also C3.2, C4.1, C5.2, C6.1, U1.2 (GND), U2.1 (GND)
